File: EggDuino77.brd (EAGLE design)
At the start: 68.6 x 53.3 mm, 27 parts

Commit message: Add GND vias
Routing:
- net VIN: track 57.2 -> 60.2 mm
Changed lines of the file:
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@@
 <contactref element="SERVO" pad="1"/>
 <contactref element="C10" pad="2"/>
+<via x="43.18" y="11.43" extent="1-16" drill="0.9" shape="octagon"/>
+<via x="48.26" y="11.43" extent="1-16" drill="0.9" shape="octagon"/>
+<via x="45.72" y="9.525" extent="1-16" drill="0.9" shape="octagon"/>
+<via x="26.67" y="13.97" extent="1-16" drill="0.9" shape="octagon"/>
+<via x="33.02" y="13.97" extent="1-16" drill="0.9" shape="octagon"/>
+<via x="29.21" y="10.795" extent="1-16" drill="0.9" shape="octagon"/>
+<via x="34.925" y="10.795" extent="1-16" drill="0.9" shape="octagon"/>
+<via x="58.42" y="8.255" extent="1-16" drill="0.9" shape="octagon"/>
+<via x="62.865" y="12.7" extent="1-16" drill="0.9" shape="octagon"/>
+<via x="33.02" y="31.115" extent="1-16" drill="0.9" shape="octagon"/>
+<via x="57.785" y="28.575" extent="1-16" drill="0.9" shape="octagon"/>
+<via x="29.21" y="44.45" extent="1-16" drill="0.9" shape="octagon"/>
+<via x="29.845" y="38.735" extent="1-16" drill="0.9" shape="octagon"/>
+<via x="56.515" y="38.735" extent="1-16" drill="0.9" shape="octagon"/>
+<via x="13.97" y="39.37" extent="1-16" drill="0.9" shape="octagon"/>
+<via x="13.97" y="45.72" extent="1-16" drill="0.9" shape="octagon"/>
+<via x="6.985" y="5.715" extent="1-16" drill="0.9" shape="octagon"/>
+<via x="61.595" y="45.085" extent="1-16" drill="0.9" shape="octagon"/>
+<via x="18.415" y="31.115" extent="1-16" drill="0.9" shape="octagon"/>
 </signal>
 <signal name="AREF" class="4">
@@
 <contactref element="C3" pad="1"/>
 <contactref element="C9" pad="1"/>
-<wire x1="45.72" y1="2.54" x2="45.72" y2="10.16" width="2.1844" layer="16"/>
-<via x="45.72" y="10.16" extent="1-16" drill="0.9" shape="octagon"/>
-<wire x1="45.72" y1="10.16" x2="41.275" y2="10.16" width="1.4224" layer="1"/>
-<wire x1="41.275" y1="10.16" x2="36.83" y2="14.605" width="1.4224" layer="1"/>
-<wire x1="36.83" y1="14.605" x2="36.83" y2="17.78" width="1.4224" layer="1"/>
-<wire x1="60.96" y1="17.78" x2="53.34" y2="10.16" width="1.4224" layer="1"/>
-<wire x1="53.34" y1="10.16" x2="45.72" y2="10.16" width="1.4224" layer="1"/>
+<wire x1="45.72" y1="2.54" x2="54.61" y2="13.97" width="2.1844" layer="16"/>
+<via x="54.61" y="13.97" extent="1-16" drill="0.9" shape="octagon"/>
+<wire x1="54.61" y1="13.97" x2="38.735" y2="13.97" width="1.4224" layer="1"/>
+<wire x1="38.735" y1="13.97" x2="36.83" y2="15.875" width="1.4224" layer="1"/>
+<wire x1="36.83" y1="15.875" x2="36.83" y2="17.78" width="1.4224" layer="1"/>
+<wire x1="60.96" y1="17.78" x2="57.15" y2="13.97" width="1.4224" layer="1"/>
+<wire x1="57.15" y1="13.97" x2="54.61" y2="13.97" width="1.4224" layer="1"/>
 <wire x1="36.83" y1="17.78" x2="36.83" y2="22.225" width="1.4224" layer="1"/>
 <wire x1="36.83" y1="22.225" x2="36.195" y2="22.86" width="1.4224" layer="1"/>
